File: kicad/pre-amp52.kicad_sch (KiCad schematic)
At the start: 70 parts, among them J1 Left, J10 L out, J11 R out, J2 LFront, J3 LRear, J4 Centre, J5 RRear, J6 RFront, J7 Right, J8 Ltape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

Commit message: Created schematic pdf and gerber files for pcb.
Parts:
- R1, R10, R11, R12, R13, R14, R15, R16, R17, R18, R19, R2, R20, R21, R22, R23, R24, R25, R26, R27, R28, R29, R3, R30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: footprint Resistor_THT:R_Axial_DIN0207_L6.3mm_D2.5mm_P10.16mm_Horizontal -> my_extras:R_Axial_DIN0207_L6.3mm_D2.5mm_P10.16mm_Horizontal
