File: kicad/untitled.kicad_sch (KiCad schematic)
At the start: 47 parts, among them J12 +12V in, J13 0V in, J14 I2C In, J15 +5V in, J16 Rpi GPIO in, K1 G6SK-2 DC12, Q1 BC546, Q2 BC546, Q3 BC546, Q4 BC556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

Commit message: Created schematic pdf and gerber files for pcb.
Parts:
- R35, R36, R37, R38, R39, R40, R41, R42, R43, R44, R45, R46: footprint Resistor_THT:R_Axial_DIN0207_L6.3mm_D2.5mm_P10.16mm_Horizontal -> my_extras:R_Axial_DIN0207_L6.3mm_D2.5mm_P10.16mm_Horizontal
Changed lines of the file:
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@@
       (effects (font (size 1.27 1.27)) (justify left))
     )
-    (property "Footprint" "Resistor_THT:R_Axial_DIN0207_L6.3mm_D2.5mm_P10.16mm_Horizontal" (id 2) (at 62.992 118.11 90)
+    (property "Footprint" "my_extras:R_Axial_DIN0207_L6.3mm_D2.5mm_P10.16mm_Horizontal" (id 2) (at 62.992 118.11 90)
       (effects (font (size 1.27 1.27)) hide)
     )
@@
       (effects (font (size 1.27 1.27)) (justify left))
     )
-    (property "Footprint" "Resistor_THT:R_Axial_DIN0207_L6.3mm_D2.5mm_P10.16mm_Horizontal" (id 2) (at 46.482 90.17 90)
+    (property "Footprint" "my_extras:R_Axial_DIN0207_L6.3mm_D2.5mm_P10.16mm_Horizontal" (id 2) (at 46.482 90.17 90)
       (effects (font (size 1.27 1.27)) hide)
     )
@@
     (property "Reference" "R38" (id 0) (at 76.2 62.3275 90))
     (property "Value" "4.7K" (id 1) (at 76.2 65.1026 90))
-    (property "Footprint" "Resistor_THT:R_Axial_DIN0207_L6.3mm_D2.5mm_P10.16mm_Horizontal" (id 2) (at 76.2 69.088 90)
+    (property "Footprint" "my_extras:R_Axial_DIN0207_L6.3mm_D2.5mm_P10.16mm_Horizontal" (id 2) (at 76.2 69.088 90)
       (effects (font (size 1.27 1.27)) hide)
     )
@@
       (effects (font (size 1.27 1.27)) (justify left))
     )
-    (property "Footprint" "Resistor_THT:R_Axial_DIN0207_L6.3mm_D2.5mm_P10.16mm_Horizontal" (id 2) (at 184.912 123.19 90)
+    (property "Footprint" "my_extras:R_Axial_DIN0207_L6.3mm_D2.5mm_P10.16mm_Horizontal" (id 2) (at 184.912 123.19 90)
       (effects (font (size 1.27 1.27)) hide)
     )
@@
       (effects (font (size 1.27 1.27)) (justify left))
     )
-    (property "Footprint" "Resistor_THT:R_Axial_DIN0207_L6.3mm_D2.5mm_P10.16mm_Horizontal" (id 2) (at 83.312 21.59 90)
+    (property "Footprint" "my_extras:R_Axial_DIN0207_L6.3mm_D2.5mm_P10.16mm_Horizontal" (id 2) (at 83.312 21.59 90)
       (effects (font (size 1.27 1.27)) hide)
     )
@@
       (effects (font (size 1.27 1.27)) hide)
     )
+    (pin "6")
+    (pin "7")
+    (pin "8")
+    (pin "10")
+    (pin "11")
+    (pin "9")
     (pin "1")
     (pin "12")
@@
       (effects (font (size 1.27 1.27)) hide)
     )
+    (pin "6")
+    (pin "7")
+    (pin "8")
+    (pin "10")
+    (pin "11")
+    (pin "9")
     (pin "1")
     (pin "12")
@@
       (effects (font (size 1.27 1.27)) hide)
     )
+    (pin "3")
+    (pin "4")
+    (pin "5")
+    (pin "10")
+    (pin "8")
+    (pin "9")
     (pin "1")
     (pin "12")
@@
       (effects (font (size 1.27 1.27)) (justify left))
     )
-    (property "Footprint" "Resistor_THT:R_Axial_DIN0207_L6.3mm_D2.5mm_P10.16mm_Horizontal" (id 2) (at 83.312 118.11 90)
+    (property "Footprint" "my_extras:R_Axial_DIN0207_L6.3mm_D2.5mm_P10.16mm_Horizontal" (id 2) (at 83.312 118.11 90)
       (effects (font (size 1.27 1.27)) hide)
     )
@@
       (effects (font (size 1.27 1.27)) hide)
     )
+    (pin "6")
+    (pin "7")
+    (pin "8")
+    (pin "10")
+    (pin "11")
+    (pin "9")
     (pin "1")
     (pin "12")
@@
       (effects (font (size 1.27 1.27)) (justify left))
     )
-    (property "Footprint" "Resistor_THT:R_Axial_DIN0207_L6.3mm_D2.5mm_P10.16mm_Horizontal" (id 2) (at 37.592 90.17 90)
+    (property "Footprint" "my_extras:R_Axial_DIN0207_L6.3mm_D2.5mm_P10.16mm_Horizontal" (id 2) (at 37.592 90.17 90)
       (effects (font (size 1.27 1.27)) hide)
     )
@@
       (effects (font (size 1.27 1.27)) (justify left))
     )
-    (property "Footprint" "Resistor_THT:R_Axial_DIN0207_L6.3mm_D2.5mm_P10.16mm_Horizontal" (id 2) (at 224.282 123.19 90)
+    (property "Footprint" "my_extras:R_Axial_DIN0207_L6.3mm_D2.5mm_P10.16mm_Horizontal" (id 2) (at 224.282 123.19 90)
       (effects (font (size 1.27 1.27)) hide)
     )
@@
       (effects (font (size 1.27 1.27)) (justify left))
     )
-    (property "Footprint" "Resistor_THT:R_Axial_DIN0207_L6.3mm_D2.5mm_P10.16mm_Horizontal" (id 2) (at 96.012 39.37 90)
+    (property "Footprint" "my_extras:R_Axial_DIN0207_L6.3mm_D2.5mm_P10.16mm_Horizontal" (id 2) (at 96.012 39.37 90)
       (effects (font (size 1.27 1.27)) hide)
     )
@@
       (effects (font (size 1.27 1.27)) (justify left))
     )
-    (property "Footprint" "Resistor_THT:R_Axial_DIN0207_L6.3mm_D2.5mm_P10.16mm_Horizontal" (id 2) (at 145.542 121.92 90)
+    (property "Footprint" "my_extras:R_Axial_DIN0207_L6.3mm_D2.5mm_P10.16mm_Horizontal" (id 2) (at 145.542 121.92 90)
       (effects (font (size 1.27 1.27)) hide)
     )
@@
       (effects (font (size 1.27 1.27)) (justify right))
     )
-    (property "Footprint" "Resistor_THT:R_Axial_DIN0207_L6.3mm_D2.5mm_P10.16mm_Horizontal" (id 2) (at 220.472 123.19 90)
+    (property "Footprint" "my_extras:R_Axial_DIN0207_L6.3mm_D2.5mm_P10.16mm_Horizontal" (id 2) (at 220.472 123.19 90)
       (effects (font (size 1.27 1.27)) hide)
     )
@@
       (effects (font (size 1.27 1.27)) (justify left))
     )
-    (property "Footprint" "Resistor_THT:R_Axial_DIN0207_L6.3mm_D2.5mm_P10.16mm_Horizontal" (id 2) (at 96.012 53.34 90)
+    (property "Footprint" "my_extras:R_Axial_DIN0207_L6.3mm_D2.5mm_P10.16mm_Horizontal" (id 2) (at 96.012 53.34 90)
       (effects (font (size 1.27 1.27)) hide)
     )
@@
       (effects (font (size 1.27 1.27)) hide)
     )
+    (pin "6")
+    (pin "7")
+    (pin "8")
+    (pin "10")
+    (pin "11")
+    (pin "9")
     (pin "1")
     (pin "12")
